File: q10keyboard-addon.kicad_pcb (KiCad board)
At the start: 2 copper layers, 65 x 60 mm, 20 parts, among them J1 Conn_02x04_Top_Bottom, J2 Conn_01x08_Female, J3 Conn_01x08_Female, J4 Conn_01x08_Female, U1 BBQ10KBD, U2 STM32F030C8Tx, X1 Badgelife_sao_connector_v169b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

Commit message: fix(pcb): keyboard connector orientation
1. The keyboard connector was in a wrong orientation,
and had to be rotated 180°.
2. Move breakout connectors away from keyboard cable
3. Reduce number of breakout GND pins from 3 to 1
4. Add ground zone below the keyboard connector to make soldering easier
Parts:
- D1, R3: moved to B.Cu
- J2: value Conn_01x08_Female -> Conn_01x06_Female; footprint Connector_PinSocket_2.54mm:PinSocket_1x08_P2.54mm_Vertical -> Connector_PinSocket_2.54mm:PinSocket_1x06_P2.54mm_Vertical
- moved R1 36.2 mm to (121.2, 65.9), turned to 90 degrees
- moved R2 36.1 mm to (122.9, 65.8), turned to 90 degrees
- moved D1 16.9 mm to (114.8, 65.8), turned to 180 degrees
- moved R3 14.5 mm to (114.8, 64.1), turned to 0 degrees
- moved JP1 11.0 mm to (138.7, 103.5), turned to 90 degrees
- moved C1 8.40 mm to (117.0, 79.4)
- moved C2 8.40 mm to (126.9, 73.0)
- moved C3 8.40 mm to (128.7, 73.0)
- moved C5 8.40 mm to (126.1, 66.1)
- moved U2 8.40 mm to (120.9, 72.6)
- moved C4 8.40 mm to (115.7, 77.6)
- moved C6 8.40 mm to (126.1, 67.9)
- moved J3 6.74 mm to (117.0, 84.6)
- moved J4 5.85 mm to (112.0, 89.8)
- moved J2 0.81 mm to (117.2, 94.8)
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Connections:
- J2 pad 2: /MIC -> /LEDA_1_2
- J2 pad 3: GNDA -> /LEDK_1_4
- J2 pad 4: /LEDK_2_3 -> /LEDA_3_4
- J2 pad 5: /LEDK_1_4 -> /LEDK_2_3
- J2 pad 6: /LEDA_3_4 -> GND
- J3 pad 1: Net-(J3-Pad1) -> GNDA
- J3 pad 6: GND -> Net-(J3-Pad6)
- J4 pad 8: GND -> /MIC
- U1 pad 10: Net-(J3-Pad3) -> Net-(J3-Pad4)
- U1 pad 17: Net-(J3-Pad4) -> Net-(J3-Pad5)
- U1 pad 19: Net-(J3-Pad5) -> Net-(J3-Pad6)
- U1 pad 7: Net-(J3-Pad1) -> Net-(J3-Pad2)
- U1 pad 9: Net-(J3-Pad2) -> Net-(J3-Pad3)
- U2 pad 17: /MIC -> Net-(U2-Pad17)
- U2 pad 29: Net-(J3-Pad5) -> Net-(J3-Pad6)
- U2 pad 30: Net-(J3-Pad4) -> Net-(J3-Pad5)
- U2 pad 31: Net-(J3-Pad3) -> Net-(J3-Pad4)
- U2 pad 32: Net-(J3-Pad2) -> Net-(J3-Pad3)
- U2 pad 33: Net-(J3-Pad1) -> Net-(J3-Pad2)
Routing:
- net Net-(J3-Pad1): track 33.2 -> 0.00 mm, vias 1 -> 0
- net GNDA: track 20.3 -> 42.1 mm, vias 1 -> 0
- net Net-(J3-Pad6): track 0.00 -> 19.6 mm, vias 0 -> 1
- net /LEDK_2_3: track 27.9 -> 10.3 mm, vias 1 -> 0
- net Net-(J3-Pad3): track 45.9 -> 30.5 mm, vias 0 -> 1
- net /MIC: track 23.7 -> 38.5 mm, vias 0 -> 1
- net Net-(J4-Pad7): track 10.6 -> 23.3 mm, vias 0 -> 1
- net Net-(J3-Pad2): track 21.7 -> 32.9 mm
- net Net-(J4-Pad3): track 37.8 -> 27.3 mm, vias 2 -> 0
- net Net-(J4-Pad1): track 34.3 -> 42.7 mm, vias 1 -> 0
- net GND: track 36.1 -> 28.3 mm, vias 1 -> 6
- net Net-(J4-Pad4): track 16.4 -> 23.7 mm, vias 1 -> 0
- net Net-(J4-Pad5): track 13.7 -> 20.4 mm, vias 1 -> 0
- net /LEDK_1_4: track 20.6 -> 14.4 mm, vias 1 -> 0
- net /LEDA_3_4: track 15.7 -> 11.8 mm, vias 1 -> 0
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- added copper zone on B.Cu, net GND
- added copper zone on F.Cu, net GND
Other:
- board text added: "R3"
- board text added: "R4"
- board text added: "R5"
- board text added: "R6"
- board text added: "R7"
- board text removed: "..."

Commit message: feat: elongate keyboard connector pads
Parts:
- U1: footprint Connectors_Hirose_extra:BM14B(0.8)-24DS-0.4V(53) -> Connectors_Hirose_extra:BM14B(0.8)-24DS-0.4V(53)-longpads
- moved JP1 31.6 mm to (113.4, 84.6), turned to 0 degrees
Routing:
- net /MIC: track 38.5 -> 41.5 mm
- net Net-(J3-Pad3): track 30.5 -> 33.1 mm
- net GNDA: track 42.1 -> 44.6 mm
- net Net-(J4-Pad3): track 27.3 -> 28.7 mm
- net Net-(J3-Pad5): track 21.5 -> 22.8 mm
- net Net-(J4-Pad1): track 42.7 -> 43.8 mm
- net /LEDA_3_4: track 11.8 -> 12.9 mm
- net Net-(J4-Pad5): track 20.4 -> 21.5 mm
- net Net-(J3-Pad2): track 32.9 -> 34.0 mm
- net Net-(J4-Pad2): track 36.5 -> 37.5 mm
- net /LEDK_2_3: track 10.3 -> 11.3 mm
- net Net-(J4-Pad4): track 23.7 -> 24.7 mm
- net Net-(J4-Pad6): track 15.9 -> 16.8 mm
- net GND: track 28.3 -> 27.8 mm, vias 6 -> 5

Commit message: feat: wire the CPU
also add reset capacitor, boot0 resistor, and round some corners
Parts:
- added C7: 100nF, Capacitor_SMD:C_0603_1608Metric, B.Cu at (127.8, 70.8)
- added R4: 10K, Resistor_SMD:R_0603_1608Metric, B.Cu at (107.3, 81.3)
- moved D1 23.9 mm to (96.7, 81.3)
- moved C1 13.3 mm to (128.7, 73.1), turned to 270 degrees
- moved C3 13.0 mm to (117.3, 79.2), turned to 0 degrees
- moved R3 4.00 mm to (118.7, 65.0)
- moved J1 1.32 mm to (106.3, 88.5)
- moved C6 1.22 mm to (125.3, 67.0), turned to 90 degrees
- moved C5 1.19 mm to (127.0, 67.0), turned to 270 degrees
- moved C2 0.15 mm to (127.0, 73.1)
- moved R1 0.10 mm to (121.2, 65.8)
Connections:
- net Net-(J4-Pad1) renamed /ROW1
- net Net-(J4-Pad2) renamed /ROW2
- net Net-(J4-Pad3) renamed /ROW3
- net Net-(J4-Pad4) renamed /ROW4
- net Net-(J4-Pad5) renamed /ROW5
- net Net-(J4-Pad6) renamed /ROW6
- net Net-(J4-Pad7) renamed /ROW7
- C1 pad 1: GND -> GNDA
- C1 pad 2: VCC -> Net-(C1-Pad2)
- C2 pad 1: VCC -> Net-(C1-Pad2)
- C2 pad 2: GND -> GNDA
- J3 pad 2: Net-(J3-Pad2) -> /COL1
- J3 pad 3: Net-(J3-Pad3) -> /COL2
- J3 pad 4: Net-(J3-Pad4) -> /COL3
- J3 pad 5: Net-(J3-Pad5) -> /COL4
- J3 pad 6: Net-(J3-Pad6) -> /COL5
- U1 pad 10: Net-(J3-Pad4) -> /COL3
- U1 pad 17: Net-(J3-Pad5) -> /COL4
- U1 pad 19: Net-(J3-Pad6) -> /COL5
- U1 pad 7: Net-(J3-Pad2) -> /COL1
- U1 pad 9: Net-(J3-Pad3) -> /COL2
- U2 pad 18: /LEDA_1_2 -> Net-(U2-Pad18)
- U2 pad 19: /LEDA_3_4 -> Net-(U2-Pad19)
- U2 pad 20: /LEDK_1_4 -> Net-(U2-Pad20)
- U2 pad 22: Net-(U2-Pad22) -> /COL5
- U2 pad 25: Net-(U2-Pad25) -> /COL4
- U2 pad 26: Net-(U2-Pad26) -> /COL3
- U2 pad 27: Net-(U2-Pad27) -> /COL2
- U2 pad 28: Net-(U2-Pad28) -> /COL1
- U2 pad 29: Net-(J3-Pad6) -> Net-(U2-Pad29)
- U2 pad 30: Net-(J3-Pad5) -> /LEDK_2_3
- U2 pad 31: Net-(J3-Pad4) -> /LEDA_3_4
- U2 pad 32: Net-(J3-Pad3) -> /LEDK_1_4
- U2 pad 33: Net-(J3-Pad2) -> /LEDA_1_2
- U2 pad 39: /LEDK_2_3 -> Net-(U2-Pad39)
- U2 pad 40: /LED -> Net-(U2-Pad40)
- U2 pad 43: Net-(U2-Pad43) -> /LED
- U2 pad 9: VCC -> Net-(C1-Pad2)
Routing:
- net VCC: track 31.1 -> 148.3 mm, vias 0 -> 2
- net /SDA: track 0.00 -> 52.8 mm, vias 0 -> 1
- net /COL1: track 0.00 -> 51.7 mm, vias 0 -> 1
- net /COL2: track 0.00 -> 50.8 mm, vias 0 -> 1
- net /SCL: track 0.00 -> 49.4 mm, vias 0 -> 1
- net /COL3: track 0.00 -> 47.4 mm, vias 0 -> 1
- net /NRST: track 0.00 -> 44.7 mm, vias 0 -> 2
- net /COL4: track 0.00 -> 43.3 mm, vias 0 -> 1
- net /TX: track 0.00 -> 43.3 mm, vias 0 -> 1
- net /LEDK_2_3: track 11.3 -> 50.2 mm
- net /LEDA_3_4: track 12.9 -> 50.5 mm
- net /LEDK_1_4: track 14.4 -> 50.5 mm
- net /ROW6: track 16.8 -> 52.1 mm, vias 0 -> 1
- net /LEDA_1_2: track 17.1 -> 51.7 mm
- net Net-(J3-Pad2): track 34.0 -> 0.00 mm, vias 1 -> 0
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Other:
- outline, holes or cut-outs redrawn

Commit message: fix: keyboard dimensions
enlarge keyboard by ~1.6%, after measuring with calipers
Parts:
- moved svg2mod 2.57 mm to (125.5, 54.4)
- moved KBD1 1.03 mm to (123.8, 76.1)
Other:
- board size 65 x 60 mm -> 65 x 63.5 mm
- board text added: "JLCJLCJLCJLC"

Commit message: feat: add 2kbit EEPROM device
The EEPROM device will be used to store the add-on id:
https://github.com/urish/badge-addon-id
Parts:
- added C8: 100nF, Capacitor_SMD:C_0603_1608Metric, B.Cu at (107.1, 69.6)
- added R5: 10K, Resistor_SMD:R_0603_1608Metric, B.Cu at (110.8, 66.9)
- added U3: M24C02-WMN, Package_SO:SOIC-8_3.9x4.9mm_P1.27mm, B.Cu at (105.5, 65.7)
Routing:
- net VCC: track 148.3 -> 165.7 mm
- net /SDA: track 52.8 -> 69.6 mm, vias 1 -> 3
- net /SCL: track 49.4 -> 64.2 mm, vias 1 -> 3
- net Net-(R5-Pad1): track 0.00 -> 2.96 mm

Commit message: fix: missing power connection for STM32 VDDA pin
Connections:
- C1 pad 2: Net-(C1-Pad2) -> VCC
- C2 pad 1: Net-(C1-Pad2) -> VCC
- U2 pad 9: Net-(C1-Pad2) -> VCC
Routing:
- net VCC: track 165.7 -> 174.1 mm
- net Net-(C1-Pad2): track 3.55 -> 0.00 mm
