File: q10keyboard-addon.kicad_pcb (KiCad board)
At the start: 2 copper layers, 65 x 63.5 mm, 25 parts, among them J1 Conn_02x04_Top_Bottom, J2 Conn_01x06_Female, J3 Conn_01x08_Female, J4 Conn_01x08_Female, U1 BBQ10KBD, U2 STM32F030C8Tx, U3 M24C02-WMN, X1 Badgelife_sao_connector_v169b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

Commit message: feat: add 3 fiducials
also move conference logo to solder mask layer
Parts:
- added REF**: Fiducial_1mm_Mask3mm, Fiducial:Fiducial_1mm_Mask3mm, B.Cu at (112.6, 103.2)
- added REF**: Fiducial_1mm_Mask3mm, Fiducial:Fiducial_1mm_Mask3mm, B.Cu at (103.4, 49.0)
- added REF**: Fiducial_1mm_Mask3mm, Fiducial:Fiducial_1mm_Mask3mm, B.Cu at (147.2, 49.0)
