File: q10keyboard-addon.sch (KiCad schematic (older format))
At the start: 18 parts, among them J1 Conn_02x04_Top_Bottom, J2 Conn_01x08_Female, J3 Conn_01x08_Female, J4 Conn_01x08_Female, U1 BBQ10KBD, U2 STM32F030C8Tx, X1 Badgelife_sao_connector_v169b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

Commit message: fix(pcb): keyboard connector orientation
1. The keyboard connector was in a wrong orientation,
and had to be rotated 180°.
2. Move breakout connectors away from keyboard cable
3. Reduce number of breakout GND pins from 3 to 1
4. Add ground zone below the keyboard connector to make soldering easier
Parts:
- removed J2: Conn_01x08_Female, Connector_PinSocket_2.54mm:PinSocket_1x08_P2.54mm_Vertical, symbol Connector:Conn_01x08_Female
- added J2: Conn_01x06_Female, Connector_PinSocket_2.54mm:PinSocket_1x06_P2.54mm_Vertical, symbol Connector:Conn_01x06_Female
Connections:
- net GND: now also J2.6 (Pin_6); no longer J3.6 (Pin_6), J4.8 (Pin_8)
- net GNDA: now also J3.1 (Pin_1)
- net LEDA_1_2: now also J2.2 (Pin_2)
- net LEDA_3_4: now also J2.4 (Pin_4)
- net LEDK_1_4: now also J2.3 (Pin_3)
- net LEDK_2_3: now also J2.5 (Pin_5)
- net MIC: now also J4.8 (Pin_8); no longer U2.17 (PA7)
- net VCC: now also J2.1 (Pin_1)
- net at U1.10 (COL3), U2.31 (PA10): now also J3.4 (Pin_4); no longer J3.3 (Pin_3)
- net at U1.17 (COL4), U2.30 (PA9): now also J3.5 (Pin_5); no longer J3.4 (Pin_4)
- net at U1.19 (COL5), U2.29 (PA8): now also J3.6 (Pin_6); no longer J3.5 (Pin_5)
- net at U1.7 (COL1), U2.33 (PA12): now also J3.2 (Pin_2); no longer J3.1 (Pin_1)
- net at U1.9 (COL2), U2.32 (PA11): now also J3.3 (Pin_3); no longer J3.2 (Pin_2)
Other:
- moved on the sheet: J3
Changed lines of the file:
@@
 Wire Wire Line
 	3950 2500 4050 2500
-Wire Wire Line
-	4550 2300 4150 2300
-Text Label 4150 2300 0    50   ~ 0
-MIC
 Text Label 2500 2500 0    50   ~ 0
 MIC
@@
 	1    0    0    -1
 $EndComp
-$Comp
-L Connector:Conn_01x06_Female J3
-U 1 1 5E179C60
-P 4200 2000
-F 0 "J3" H 4100 2550 50  0000 L CNN
-F 1 "Conn_01x08_Female" H 3800 2450 50  0000 L CNN
-F 2 "Connector_PinSocket_2.54mm:PinSocket_1x06_P2.54mm_Vertical" H 4200 2000 50  0001 C CNN
-F 3 "~" H 4200 2000 50  0001 C CNN
-	1    4200 2000
-	1    0    0    -1
-$EndComp
-$Comp
-L power:GND #PWR0115
-U 1 1 5E17A5A3
-P 3900 3200
-F 0 "#PWR0115" H 3900 2950 50  0001 C CNN
-F 1 "GND" H 3905 3027 50  0000 C CNN
-F 2 "" H 3900 3200 50  0001 C CNN
-F 3 "" H 3900 3200 50  0001 C CNN
-	1    3900 3200
-	1    0    0    -1
-$EndComp
 Connection ~ 4050 2400
 Wire Wire Line
@@
 	4050 3000 4550 3000
 Wire Wire Line
-	4050 3100 3900 3100
+	4050 3100 3850 3100
 Wire Wire Line
 	3950 1800 4000 1800
@@
 Wire Wire Line
 	3950 2400 4050 2400
-Wire Wire Line
-	3900 2300 4000 2300
-Wire Wire Line
-	3900 2300 3900 3100
-Connection ~ 3900 3100
-Wire Wire Line
-	3900 3100 3900 3200
-$Comp
-L Connector:Conn_01x08_Female J2
-U 1 1 5E19B2D6
-P 2000 2300
-F 0 "J2" H 1850 1800 50  0000 L CNN
-F 1 "Conn_01x08_Female" H 1750 1700 50  0000 L CNN
-F 2 "Connector_PinSocket_2.54mm:PinSocket_1x08_P2.54mm_Vertical" H 2000 2300 50  0001 C CNN
-F 3 "~" H 2000 2300 50  0001 C CNN
-	1    2000 2300
-	-1   0    0    1
-$EndComp
 $Comp
 L power:GNDA #PWR0116
 U 1 1 5E1A7254
-P 2400 2400
-F 0 "#PWR0116" H 2400 2150 50  0001 C CNN
-F 1 "GNDA" V 2405 2273 50  0000 R CNN
-F 2 "" H 2400 2400 50  0001 C CNN
-F 3 "" H 2400 2400 50  0001 C CNN
-	1    2400 2400
-	0    -1   -1   0
+P 3700 1600
+F 0 "#PWR0116" H 3700 1350 50  0001 C CNN
+F 1 "GNDA" V 3705 1473 50  0000 R CNN
+F 2 "" H 3700 1600 50  0001 C CNN
+F 3 "" H 3700 1600 50  0001 C CNN
+	1    3700 1600
+	-1   0    0    1
 $EndComp
 Wire Wire Line
 	2600 1800 2750 1800
-$Comp
-L power:GND #PWR0117
-U 1 1 5E1B7DC3
-P 2300 1800
-F 0 "#PWR0117" H 2300 1550 50  0001 C CNN
-F 1 "GND" H 2305 1627 50  0000 C CNN
-F 2 "" H 2300 1800 50  0001 C CNN
-F 3 "" H 2300 1800 50  0001 C CNN
-	1    2300 1800
-	-1   0    0    1
-$EndComp
-Wire Wire Line
-	2300 1800 2300 1900
-Wire Wire Line
-	2300 1900 2200 1900
-Wire Wire Line
-	2200 2000 2750 2000
-Wire Wire Line
-	2200 2100 2750 2100
-Wire Wire Line
-	2200 2200 2750 2200
-Wire Wire Line
-	2200 2300 2750 2300
-Wire Wire Line
-	2200 2400 2400 2400
-Wire Wire Line
-	2200 2500 2750 2500
+Wire Wire Line
+	2300 2000 2750 2000
+Wire Wire Line
+	2300 2100 2750 2100
+Wire Wire Line
+	2300 2200 2750 2200
+Wire Wire Line
+	2300 2300 2750 2300
+Wire Wire Line
+	2500 2500 2750 2500
 $Comp
 L power:VCC #PWR0118
 U 1 1 5E1A2395
-P 2400 2600
-F 0 "#PWR0118" H 2400 2450 50  0001 C CNN
-F 1 "VCC" V 2417 2728 50  0000 L CNN
-F 2 "" H 2400 2600 50  0001 C CNN
-F 3 "" H 2400 2600 50  0001 C CNN
-	1    2400 2600
+P 1600 3500
+F 0 "#PWR0118" H 1600 3350 50  0001 C CNN
+F 1 "VCC" V 1617 3628 50  0000 L CNN
+F 2 "" H 1600 3500 50  0001 C CNN
+F 3 "" H 1600 3500 50  0001 C CNN
+	1    1600 3500
 	0    1    1    0
 $EndComp
-Wire Wire Line
-	2400 2600 2200 2600
+Text Label 1900 3400 2    50   ~ 0
+LEDA_1_2
+Text Label 1900 3200 2    50   ~ 0
+LEDA_3_4
+Text Label 1900 3300 2    50   ~ 0
+LEDK_1_4
+Text Label 1900 3100 2    50   ~ 0
+LEDK_2_3
+$Comp
+L power:GND #PWR0117
+U 1 1 5E2BFA6D
+P 1550 2900
+F 0 "#PWR0117" H 1550 2650 50  0001 C CNN
+F 1 "GND" H 1555 2727 50  0000 C CNN
+F 2 "" H 1550 2900 50  0001 C CNN
+F 3 "" H 1550 2900 50  0001 C CNN
+	1    1550 2900
+	-1   0    0    1
+$EndComp
+Wire Wire Line
+	1550 2900 1550 3000
+Wire Wire Line
+	1550 3000 1450 3000
+Wire Wire Line
+	1450 3100 1900 3100
+Wire Wire Line
+	1450 3200 1900 3200
+Wire Wire Line
+	1450 3300 1900 3300
+Wire Wire Line
+	1450 3400 1900 3400
+Text Label 3850 3100 0    50   ~ 0
+MIC
+$Comp
+L Connector:Conn_01x06_Female J3
+U 1 1 5E179C60
+P 4200 1900
+F 0 "J3" H 4100 2450 50  0000 L CNN
+F 1 "Conn_01x08_Female" H 3800 2350 50  0000 L CNN
+F 2 "Connector_PinSocket_2.54mm:PinSocket_1x06_P2.54mm_Vertical" H 4200 1900 50  0001 C CNN
+F 3 "~" H 4200 1900 50  0001 C CNN
+	1    4200 1900
+	1    0    0    -1
+$EndComp
+$Comp
+L Connector:Conn_01x06_Female J2
+U 1 1 5E32BA69
+P 1250 3300
+F 0 "J2" H 1150 3850 50  0000 L CNN
+F 1 "Conn_01x06_Female" H 850 3750 50  0000 L CNN
+F 2 "Connector_PinSocket_2.54mm:PinSocket_1x06_P2.54mm_Vertical" H 1250 3300 50  0001 C CNN
+F 3 "~" H 1250 3300 50  0001 C CNN
+	1    1250 3300
+	-1   0    0    1
+$EndComp
+Wire Wire Line
+	1600 3500 1450 3500
+Wire Wire Line
+	4000 1600 3700 1600
+Wire Wire Line
+	4000 1700 4000 1600
 $EndSCHEMATC

Commit message: feat: elongate keyboard connector pads
Parts:
- U1: footprint Connectors_Hirose_extra:BM14B(0.8)-24DS-0.4V(53) -> Connectors_Hirose_extra:BM14B(0.8)-24DS-0.4V(53)-longpads
Changed lines of the file:
@@
 F 0 "U1" H 3350 3287 60  0000 C CNN
 F 1 "BBQ10KBD" H 3350 3181 60  0000 C CNN
-F 2 "Connectors_Hirose_extra:BM14B(0.8)-24DS-0.4V(53)" H 3350 2050 60  0001 C CNN
+F 2 "Connectors_Hirose_extra:BM14B(0.8)-24DS-0.4V(53)-longpads" H 3350 2050 60  0001 C CNN
 F 3 "" H 3350 2050 60  0001 C CNN
 	1    3350 2400

Commit message: feat: wire the CPU
also add reset capacitor, boot0 resistor, and round some corners
Parts:
- added C7: 100nF, Capacitor_SMD:C_0603_1608Metric, symbol Device:C
- added R4: 10K, Resistor_SMD:R_0603_1608Metric, symbol Device:R
Connections:
- net BOOT0: now also R4.1
- net GND: now also C7.1, R4.2; no longer C1.1, C2.2
- net GNDA: now also C1.1, C2.2
- net LED: now also U2.43 (PB7); no longer U2.40 (PB4)
- net LEDA_1_2: now also U2.33 (PA12); no longer U2.18 (PB0)
- net LEDA_3_4: now also U2.31 (PA10); no longer U2.19 (PB1)
- net LEDK_1_4: now also U2.32 (PA11); no longer U2.20 (PB2)
- net LEDK_2_3: now also U2.30 (PA9); no longer U2.39 (PB3)
- net NRST: now also C7.2
- net VCC: no longer C1.2, C2.1, U2.9 (VDDA)
- net COL3: now reaches J3.4 (Pin_4), U1.10 (COL3)
- net COL3: now also U2.26 (PB13); no longer U2.31 (PA10)
- net COL4: now reaches J3.5 (Pin_5), U1.17 (COL4)
- net COL4: now also U2.25 (PB12); no longer U2.30 (PA9)
- net ROW3: now reaches J4.3 (Pin_3), U1.18 (ROW3), U2.14 (PA4)
- net COL5: now reaches J3.6 (Pin_6), U1.19 (COL5)
- net COL5: now also U2.22 (PB11); no longer U2.29 (PA8)
- net ROW4: now reaches J4.4 (Pin_4), U1.20 (ROW4), U2.13 (PA3)
- net ROW5: now reaches J4.5 (Pin_5), U1.21 (ROW5), U2.12 (PA2)
- net ROW6: now reaches J4.6 (Pin_6), U1.22 (ROW6), U2.11 (PA1)
- net ROW7: now reaches J4.7 (Pin_7), U1.27 (ROW7), U2.10 (PA0)
- net ROW1: now reaches J4.1 (Pin_1), U1.6 (ROW1), U2.16 (PA6)
- net COL1: now reaches J3.2 (Pin_2), U1.7 (COL1)
- net COL1: now also U2.28 (PB15); no longer U2.33 (PA12)
- net ROW2: now reaches J4.2 (Pin_2), U1.8 (ROW2), U2.15 (PA5)
- net COL2: now reaches J3.3 (Pin_3), U1.9 (COL2)
- net COL2: now also U2.27 (PB14); no longer U2.32 (PA11)
- new net: C1.2, C2.1, U2.9 (VDDA)
- no-connect marks 18 -> 19
Other:
- moved on the sheet: J2, J3, J4, U1

Commit message: feat: prepare for SMT assembly
Parts:
- R1: LCSC Part (none) -> C25804
- U2: LCSC Part (none) -> C23922
Changed lines of the file:
@@
 F 2 "Package_QFP:LQFP-48_7x7mm_P0.5mm" H 4650 1400 50  0001 R CNN
 F 3 "http://www.st.com/st-web-ui/static/active/en/resource/technical/document/datasheet/DM00088500.pdf" H 5150 2900 50  0001 C CNN
+F 4 "C23922" H 5150 2900 50  0001 C CNN "LCSC Part"
 	1    5150 2900
 	-1   0    0    1
@@
 F 2 "Resistor_SMD:R_0603_1608Metric" V 9280 1900 50  0001 C CNN
 F 3 "~" H 9350 1900 50  0001 C CNN
+F 4 "C25804" H 9350 1900 50  0001 C CNN "LCSC Part"
 	1    9350 1900
 	-1   0    0    1

Commit message: feat: add 2kbit EEPROM device
The EEPROM device will be used to store the add-on id:
https://github.com/urish/badge-addon-id
Parts:
- added C8: 100nF, Capacitor_SMD:C_0603_1608Metric, symbol Device:C
- added R5: 10K, Resistor_SMD:R_0603_1608Metric, symbol Device:R
- added U3: M24C02-WMN, Package_SO:SOIC-8_3.9x4.9mm_P1.27mm, symbol Memory_EEPROM:M24C02-WMN
Connections:
- net GND: now also C8.2, U3.4 (VSS)
- net SCL: now also U3.6 (SCL)
- net SDA: now also U3.5 (SDA)
- net VCC: now also C8.1, R5.2, U3.8 (VCC)
- new net: R5.1, U3.7 (~WC)
- no-connect marks 19 -> 22
Changed lines of the file:
@@
 	6450 4100 6450 4300
 Connection ~ 6450 4300
+$Comp
+L Memory_EEPROM:M24C02-WMN U3
+U 1 1 5E2DE0AD
+P 2300 1650
+F 0 "U3" H 2100 1900 50  0000 C CNN
+F 1 "M24C02-WMN" H 2250 1300 50  0000 C CNN
+F 2 "Package_SO:SOIC-8_3.9x4.9mm_P1.27mm" H 2300 2000 50  0001 C CNN
+F 3 "http://www.st.com/content/ccc/resource/technical/document/datasheet/b0/d8/50/40/5a/85/49/6f/DM00071904.pdf/files/DM00071904.pdf/jcr:content/translations/en.DM00071904.pdf" H 2350 1150 50  0001 C CNN
+F 4 "C7562" H 2300 1650 50  0001 C CNN "LCSC Part"
+	1    2300 1650
+	1    0    0    -1
+$EndComp
+Text Label 2900 1550 2    50   ~ 0
+SDA
+Wire Wire Line
+	2900 1550 2700 1550
+Text Label 2900 1650 2    50   ~ 0
+SCL
+Wire Wire Line
+	2900 1650 2700 1650
+$Comp
+L Device:C C8
+U 1 1 5E2EC355
+P 2050 1100
+F 0 "C8" H 2050 1200 50  0000 L CNN
+F 1 "100nF" H 2050 1000 50  0000 L CNN
+F 2 "Capacitor_SMD:C_0603_1608Metric" H 2088 950 50  0001 C CNN
+F 3 "~" H 2050 1100 50  0001 C CNN
+F 4 "C14663" H 2050 1100 50  0001 C CNN "LCSC Part"
+	1    2050 1100
+	0    1    1    0
+$EndComp
+Wire Wire Line
+	2200 1100 2300 1100
+Wire Wire Line
+	2300 1100 2300 1350
+$Comp
+L power:GND #PWR0120
+U 1 1 5E2F4C3E
+P 2300 2050
+F 0 "#PWR0120" H 2300 1800 50  0001 C CNN
+F 1 "GND" V 2305 1922 50  0000 R CNN
+F 2 "" H 2300 2050 50  0001 C CNN
+F 3 "" H 2300 2050 50  0001 C CNN
+	1    2300 2050
+	1    0    0    -1
+$EndComp
+Wire Wire Line
+	2300 2050 2300 1950
+$Comp
+L power:GND #PWR0121
+U 1 1 5E2FC076
+P 1800 1150
+F 0 "#PWR0121" H 1800 900 50  0001 C CNN
+F 1 "GND" V 1805 1022 50  0000 R CNN
+F 2 "" H 1800 1150 50  0001 C CNN
+F 3 "" H 1800 1150 50  0001 C CNN
+	1    1800 1150
+	1    0    0    -1
+$EndComp
+Wire Wire Line
+	1800 1100 1800 1150
+Wire Wire Line
+	1800 1100 1900 1100
+NoConn ~ 1900 1550
+NoConn ~ 1900 1650
+NoConn ~ 1900 1750
+$Comp
+L Device:R R5
+U 1 1 5E31E5D0
+P 2950 1750
+F 0 "R5" V 2850 1800 50  0000 R CNN
+F 1 "10K" V 2950 1800 50  0000 R CNN
+F 2 "Resistor_SMD:R_0603_1608Metric" V 2880 1750 50  0001 C CNN
+F 3 "~" H 2950 1750 50  0001 C CNN
+F 4 "C25804" H 2950 1750 50  0001 C CNN "LCSC Part"
+	1    2950 1750
+	0    -1   -1   0
+$EndComp
+Wire Wire Line
+	2700 1750 2800 1750
+$Comp
+L power:VCC #PWR0122
+U 1 1 5E326184
+P 2300 900
+F 0 "#PWR0122" H 2300 750 50  0001 C CNN
+F 1 "VCC" V 2318 1027 50  0000 L CNN
+F 2 "" H 2300 900 50  0001 C CNN
+F 3 "" H 2300 900 50  0001 C CNN
+	1    2300 900
+	0    1    1    0
+$EndComp
+Wire Wire Line
+	2300 900  2300 1100
+Connection ~ 2300 1100
+$Comp
+L power:VCC #PWR0123
+U 1 1 5E32EECF
+P 3200 1750
+F 0 "#PWR0123" H 3200 1600 50  0001 C CNN
+F 1 "VCC" V 3218 1877 50  0000 L CNN
+F 2 "" H 3200 1750 50  0001 C CNN
+F 3 "" H 3200 1750 50  0001 C CNN
+	1    3200 1750
+	0    1    1    0
+$EndComp
+Wire Wire Line
+	3200 1750 3100 1750
 $EndSCHEMATC

Commit message: fix: missing power connection for STM32 VDDA pin
Connections:
- net VCC: now also C1.2, C2.1, U2.9 (VDDA)
Changed lines of the file:
@@
 $EndComp
 Wire Wire Line
-	8750 4250 9000 4250
+	8750 4250 8900 4250
 $Comp
 L power:GND #PWR0107
 U 1 1 5E15817A
-P 10300 4400
-F 0 "#PWR0107" H 10300 4150 50  0001 C CNN
-F 1 "GND" H 10305 4227 50  0000 C CNN
-F 2 "" H 10300 4400 50  0001 C CNN
-F 3 "" H 10300 4400 50  0001 C CNN
-	1    10300 4400
-	1    0    0    -1
-$EndComp
-Wire Wire Line
-	10100 4250 10300 4250
-Wire Wire Line
-	10300 4250 10300 4400
+P 10500 4250
+F 0 "#PWR0107" H 10500 4000 50  0001 C CNN
+F 1 "GND" H 10505 4077 50  0000 C CNN
+F 2 "" H 10500 4250 50  0001 C CNN
+F 3 "" H 10500 4250 50  0001 C CNN
+	1    10500 4250
+	1    0    0    -1
+$EndComp
+Wire Wire Line
+	10100 4250 10150 4250
 Text Label 8750 4050 0    50   ~ 0
 SDA
@@
 Wire Wire Line
 	6050 2100 5750 2100
-Wire Wire Line
-	4550 1800 4100 1800
 Text Label 4100 1800 0    50   ~ 0
 LEDA_1_2
@@
 Text Label 4100 2000 0    50   ~ 0
 LEDA_3_4
-Wire Wire Line
-	4550 1900 4100 1900
 Text Label 1100 5850 0    50   ~ 0
 LEDK_1_4
 Text Label 4100 1900 0    50   ~ 0
 LEDK_1_4
-Wire Wire Line
-	4550 2000 4100 2000
 Text Label 1100 5950 0    50   ~ 0
 LEDK_2_3
 Text Label 4100 2100 0    50   ~ 0
 LEDK_2_3
-Wire Wire Line
-	4100 2100 4550 2100
 NoConn ~ 5750 2000
 NoConn ~ 5750 3200
@@
 Wire Wire Line
 	1400 5450 1550 5450
-Wire Wire Line
-	1100 5650 1550 5650
 Wire Wire Line
 	1100 5750 1550 5750
@@
 Wire Wire Line
 	3200 1750 3100 1750
+$Comp
+L power:PWR_FLAG #FLG0101
+U 1 1 5E344D62
+P 8900 4250
+F 0 "#FLG0101" H 8900 4325 50  0001 C CNN
+F 1 "PWR_FLAG" H 8900 4423 50  0000 C CNN
+F 2 "" H 8900 4250 50  0001 C CNN
+F 3 "~" H 8900 4250 50  0001 C CNN
+	1    8900 4250
+	-1   0    0    1
+$EndComp
+Connection ~ 8900 4250
+Wire Wire Line
+	8900 4250 9000 4250
+$Comp
+L power:PWR_FLAG #FLG0102
+U 1 1 5E3458F1
+P 10150 4250
+F 0 "#FLG0102" H 10150 4325 50  0001 C CNN
+F 1 "PWR_FLAG" H 10150 4423 50  0000 C CNN
+F 2 "" H 10150 4250 50  0001 C CNN
+F 3 "~" H 10150 4250 50  0001 C CNN
+	1    10150 4250
+	-1   0    0    1
+$EndComp
+Connection ~ 10150 4250
+Wire Wire Line
+	10150 4250 10500 4250
+Wire Wire Line
+	4750 4900 5000 4900
+Connection ~ 5000 4900
+Wire Wire Line
+	4100 2100 4550 2100
+Wire Wire Line
+	4550 2000 4100 2000
+Wire Wire Line
+	4550 1900 4100 1900
+Wire Wire Line
+	4550 1800 4100 1800
+Wire Wire Line
+	1100 5650 1550 5650
+$Comp
+L power:PWR_FLAG #FLG0103
+U 1 1 5E38A937
+P 7950 1900
+F 0 "#FLG0103" H 7950 1975 50  0001 C CNN
+F 1 "PWR_FLAG" V 7950 2028 50  0000 L CNN
+F 2 "" H 7950 1900 50  0001 C CNN
+F 3 "~" H 7950 1900 50  0001 C CNN
+	1    7950 1900
+	0    1    1    0
+$EndComp
+Wire Wire Line
+	7950 1900 7800 1900
+Connection ~ 7800 1900
 $EndSCHEMATC
